File: ModuCard-System-ActiveBackplane/CH334R.kicad_sch (KiCad schematic)
At the start: 6 parts, among them U4 CH334R, Y4 12MHz

Commit message: [2][5] Aplly layout finishing touches
Parts:
- renumbered C20 to C13, C21 to C14, C23 to C15, C24 to C16
Connections:
- net USB1.+: now also U4.2 (DP4); no longer U4.8 (DP1)
- net USB1.-: now also U4.1 (DM4); no longer U4.7 (DM1)
- net USB2.+: now also U4.4 (DP3); no longer U4.6 (DP2)
- net USB2.-: now also U4.3 (DM3); no longer U4.5 (DM2)
- net USB3.+: now also U4.6 (DP2); no longer U4.4 (DP3)
- net USB3.-: now also U4.5 (DM2); no longer U4.3 (DM3)
- net USB4.+: now also U4.8 (DP1); no longer U4.2 (DP4)
- net USB4.-: now also U4.7 (DM1); no longer U4.1 (DM4)
