File: ModuCard-System-ActiveBackplane/Connector.kicad_sch (KiCad schematic)
At the start: 1 part, among them J4 09031967921

Commit message: [2][5] Aplly layout finishing touches
Connections:
- net USB.+: now also J4.a2; no longer J4.c2
- net USB.-: now also J4.c2; no longer J4.a2
