File: ModuCard-System-ActiveBackplane/ModuCard-System-ActiveBackplane.kicad_sch (KiCad schematic)
At the start: 8 parts

Commit message: [2][5] Aplly layout finishing touches
Parts:
- renumbered D3 to D1, D1 to D3, NT17 to NT1, NT18 to NT2, R6 to R1, R5 to R2, R11 to R3
Connections:
- net USBIN.+: now also NT2.1; no longer NT1.1
- net USBIN.-: now also NT1.1; no longer NT2.1
Changed lines of the file:
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@@
 	)
 	(label "USBIN.+"
-		(at 176.53 124.46 0)
+		(at 176.53 128.27 0)
 		(fields_autoplaced yes)
 		(effects
@@
 	)
 	(label "USBIN.-"
-		(at 176.53 128.27 0)
+		(at 176.53 124.46 0)
 		(fields_autoplaced yes)
 		(effects
@@
 		(on_board yes)
 		(dnp no)
-		(property "Reference" "#PWR09"
+		(property "Reference" "#PWR01"
 			(at 27.94 97.79 0)
 			(effects
@@
 			(project "ModuCard-System-ActiveBackplane"
 				(path "/8ab7bab9-e078-4eba-84b5-91e80d010216"
-					(reference "#PWR09")
+					(reference "#PWR01")
 					(unit 1)
 				)
@@
 		(on_board yes)
 		(dnp no)
-		(property "Reference" "R6"
+		(property "Reference" "R1"
 			(at 30.226 110.744 90)
 			(effects
@@
 			(project "ModuCard-System-ActiveBackplane"
 				(path "/8ab7bab9-e078-4eba-84b5-91e80d010216"
-					(reference "R6")
+					(reference "R1")
 					(unit 1)
 				)
@@
 		(on_board yes)
 		(dnp no)
-		(property "Reference" "R11"
+		(property "Reference" "R3"
 			(at 53.086 110.744 90)
 			(effects
@@
 			(project "ModuCard-System-ActiveBackplane"
 				(path "/8ab7bab9-e078-4eba-84b5-91e80d010216"
-					(reference "R11")
+					(reference "R3")
 					(unit 1)
 				)
@@
 		(on_board yes)
 		(dnp no)
-		(property "Reference" "#PWR0631"
+		(property "Reference" "#PWR03"
 			(at 50.8 97.79 0)
 			(effects
@@
 			(project "ModuCard-System-ActiveBackplane"
 				(path "/8ab7bab9-e078-4eba-84b5-91e80d010216"
-					(reference "#PWR0631")
+					(reference "#PWR03")
 					(unit 1)
 				)
@@
 		(on_board yes)
 		(dnp no)
-		(property "Reference" "#PWR012"
+		(property "Reference" "#PWR06"
 			(at 50.8 139.7 0)
 			(effects
@@
 			(project "ModuCard-System-ActiveBackplane"
 				(path "/8ab7bab9-e078-4eba-84b5-91e80d010216"
-					(reference "#PWR012")
+					(reference "#PWR06")
 					(unit 1)
 				)
@@
 		(on_board yes)
 		(dnp no)
-		(property "Reference" "D3"
+		(property "Reference" "D1"
 			(at 30.734 118.618 0)
 			(effects
@@
 			(project "ModuCard-System-ActiveBackplane"
 				(path "/8ab7bab9-e078-4eba-84b5-91e80d010216"
-					(reference "D3")
+					(reference "D1")
 					(unit 1)
 				)
@@
 		(on_board yes)
 		(dnp no)
-		(property "Reference" "#PWR06"
+		(property "Reference" "#PWR05"
 			(at 39.37 139.7 0)
 			(effects
@@
 			(project "ModuCard-System-ActiveBackplane"
 				(path "/8ab7bab9-e078-4eba-84b5-91e80d010216"
-					(reference "#PWR06")
+					(reference "#PWR05")
 					(unit 1)
 				)
@@
 		(on_board yes)
 		(dnp no)
-		(property "Reference" "#PWR05"
+		(property "Reference" "#PWR02"
 			(at 39.37 97.79 0)
 			(effects
@@
 			(project "ModuCard-System-ActiveBackplane"
 				(path "/8ab7bab9-e078-4eba-84b5-91e80d010216"
-					(reference "#PWR05")
+					(reference "#PWR02")
 					(unit 1)
 				)
@@
 		(on_board yes)
 		(dnp no)
-		(property "Reference" "NT17"
+		(property "Reference" "NT1"
 			(at 187.706 125.476 0)
 			(effects
@@
 			(project "ModuCard-System-ActiveBackplane"
 				(path "/8ab7bab9-e078-4eba-84b5-91e80d010216"
-					(reference "NT17")
+					(reference "NT1")
 					(unit 1)
 				)
@@
 		(on_board yes)
 		(dnp no)
-		(property "Reference" "#PWR010"
+		(property "Reference" "#PWR04"
 			(at 27.94 139.7 0)
 			(effects
@@
 			(project "ModuCard-System-ActiveBackplane"
 				(path "/8ab7bab9-e078-4eba-84b5-91e80d010216"
-					(reference "#PWR010")
+					(reference "#PWR04")
 					(unit 1)
 				)
@@
 		(on_board yes)
 		(dnp no)
-		(property "Reference" "NT18"
+		(property "Reference" "NT2"
 			(at 187.706 129.54 0)
 			(effects
@@
 			(project "ModuCard-System-ActiveBackplane"
 				(path "/8ab7bab9-e078-4eba-84b5-91e80d010216"
-					(reference "NT18")
+					(reference "NT2")
 					(unit 1)
 				)
@@
 		(on_board yes)
 		(dnp no)
-		(property "Reference" "R5"
+		(property "Reference" "R2"
 			(at 41.656 110.744 90)
 			(effects
@@
 			(project "ModuCard-System-ActiveBackplane"
 				(path "/8ab7bab9-e078-4eba-84b5-91e80d010216"
-					(reference "R5")
+					(reference "R2")
 					(unit 1)
 				)
@@
 		(on_board yes)
 		(dnp no)
-		(property "Reference" "D1"
+		(property "Reference" "D3"
 			(at 53.594 118.618 0)
 			(effects
@@
 			(project "ModuCard-System-ActiveBackplane"
 				(path "/8ab7bab9-e078-4eba-84b5-91e80d010216"
-					(reference "D1")
-					(unit 1)
-				)
+					(reference "D3")
+					(unit 1)
+				)
