File: ModuCard-System-ActiveBackplane/Mounting holes.kicad_sch (KiCad schematic)
At the start: 36 parts

Commit message: [2][5] Aplly layout finishing touches
Parts:
- renumbered H16 to H15, H17 to H16, H18 to H17, H21 to H18, H22 to H19, H23 to H20, H24 to H21, H25 to H22, H26 to H23, H27 to H24, H28 to H25, H29 to H26, H30 to H27, H31 to H28, H32 to H29, H33 to H30, H34 to H31, H35 to H32, H36 to H33, H37 to H34, H38 to H35, H39 to H36
