File: ModuCard-System-ActiveBackplane/CanTerminators.kicad_sch (KiCad schematic)
At the start: 14 parts, among them SW1 SW_DIP_x02, SW2 SW_DIP_x02

Commit message: [2][5] Aplly layout finishing touches
Parts:
- renumbered C1 to C21, C2 to C22, C3 to C23, C4 to C24, R9 to R11, R2 to R4, R1 to R5, R4 to R6, R3 to R7, R7 to R9
Other:
- moved on the sheet: C21, C22, C23, C24, R10, R11, R4, R5, R6, R7, R8, R9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

Commit message: [2][1][5] Add via stitching, fix net tie footprint
Connections:
- net at R5.1, SW1.1: no longer names the net of R5.1, SW1.1
- net at R5.1, SW1.1: no longer R9.1, SW1.2
- new net: R9.1, SW1.2
Changed lines of the file:
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@@
 	(wire
 		(pts
-			(xy 22.86 107.95) (xy 19.05 107.95)
+			(xy 45.72 107.95) (xy 40.64 107.95)
 		)
 		(stroke
@@
 	(wire
 		(pts
-			(xy 227.33 97.79) (xy 229.87 97.79)
+			(xy 22.86 107.95) (xy 19.05 107.95)
 		)
 		(stroke
@@
 	(wire
 		(pts
-			(xy 67.31 97.79) (xy 64.77 97.79)
+			(xy 227.33 97.79) (xy 229.87 97.79)
 		)
 		(stroke
@@
 	(wire
 		(pts
-			(xy 275.59 82.55) (xy 275.59 68.58)
+			(xy 67.31 97.79) (xy 64.77 97.79)
 		)
 		(stroke
@@
 	(wire
 		(pts
-			(xy 45.72 107.95) (xy 40.64 107.95)
+			(xy 275.59 82.55) (xy 275.59 68.58)
 		)
 		(stroke
@@
 	(wire
 		(pts
-			(xy 45.72 82.55) (xy 45.72 95.25)
+			(xy 30.48 107.95) (xy 31.75 107.95)
 		)
 		(stroke
@@
 	(wire
 		(pts
-			(xy 30.48 107.95) (xy 31.75 107.95)
+			(xy 271.78 107.95) (xy 275.59 107.95)
 		)
 		(stroke
@@
 	(wire
 		(pts
-			(xy 271.78 107.95) (xy 275.59 107.95)
+			(xy 49.53 97.79) (xy 45.72 97.79)
 		)
 		(stroke
@@
 	(wire
 		(pts
-			(xy 45.72 95.25) (xy 49.53 95.25)
-		)
-		(stroke
-			(width 0)
-			(type default)
-		)
-	)
-	(wire
-		(pts
 			(xy 245.11 95.25) (xy 250.19 95.25)
 		)
@@
 	(wire
 		(pts
-			(xy 45.72 97.79) (xy 45.72 107.95)
+			(xy 67.31 95.25) (xy 64.77 95.25)
 		)
 		(stroke
@@
 	(wire
 		(pts
-			(xy 67.31 95.25) (xy 64.77 95.25)
+			(xy 97.79 48.26) (xy 200.66 48.26)
 		)
 		(stroke
@@
 	(wire
 		(pts
-			(xy 49.53 97.79) (xy 45.72 97.79)
+			(xy 19.05 82.55) (xy 19.05 68.58)
 		)
 		(stroke
@@
 	(wire
 		(pts
-			(xy 97.79 48.26) (xy 200.66 48.26)
+			(xy 262.89 116.84) (xy 262.89 115.57)
 		)
 		(stroke
@@
 		)
 	)
-	(wire
+	(bus
 		(pts
-			(xy 19.05 82.55) (xy 19.05 68.58)
+			(xy 95.25 48.26) (xy 95.25 50.8)
 		)
 		(stroke
@@
 	(wire
 		(pts
-			(xy 262.89 116.84) (xy 262.89 115.57)
+			(xy 31.75 107.95) (xy 33.02 107.95)
 		)
 		(stroke
@@
 		)
 	)
-	(bus
+	(wire
 		(pts
-			(xy 95.25 48.26) (xy 95.25 50.8)
+			(xy 45.72 95.25) (xy 49.53 95.25)
 		)
 		(stroke
@@
 	(wire
 		(pts
-			(xy 31.75 107.95) (xy 33.02 107.95)
+			(xy 31.75 91.44) (xy 31.75 90.17)
 		)
 		(stroke
@@
 	(wire
 		(pts
-			(xy 31.75 91.44) (xy 31.75 90.17)
+			(xy 45.72 82.55) (xy 45.72 95.25)
 		)
 		(stroke
@@
 	(wire
 		(pts
+			(xy 45.72 97.79) (xy 45.72 107.95)
+		)
+		(stroke
+			(width 0)
+			(type default)
+		)
+	)
+	(wire
+		(pts
 			(xy 245.11 97.79) (xy 250.19 97.79)
 		)
@@
 		)
 	)
-	(label ""
-		(at 49.53 95.25 0)
-		(fields_autoplaced yes)
-		(effects
-			(font
-				(size 1.27 1.27)
-			)
-			(justify left bottom)
-		)
-	)
 	(label "CAN1.-"
 		(at 115.57 31.75 180)
@@
 		)
 	)
-	(label ""
-		(at 49.53 97.79 180)
-		(fields_autoplaced yes)
-		(effects
-			(font
-				(size 1.27 1.27)
-			)
-			(justify right bottom)
-		)
-	)
